File: KiCAD/BLDC_STC15W401.kicad_pcb (KiCad board)
At the start: 2 copper layers, 65 x 50 mm, 55 parts, among them J1 Download, J2 PPM, J3 BLDC, J4 DC12V, J5 DC5V, J6 PWM, J7 BLDC, Q1 DTC143Z, Q2 Q_PMOS_GSD, Q3 Q_NMOS_GSD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

Commit message: 添加V0.2的PCB设计
Parts:
- added Q10: Q_NMOS_GDS, TO_SOT_Packages_SMD:TO-252-2, F.Cu at (123.0, 49.0)
- added Q11: Q_NMOS_GDS, TO_SOT_Packages_SMD:TO-252-2, F.Cu at (123.0, 58.0)
- added Q12: Q_NMOS_GDS, TO_SOT_Packages_SMD:TO-252-2, F.Cu at (123.0, 67.0)
- added Q13: Q_NMOS_GDS, TO_SOT_Packages_SMD:TO-252-2, F.Cu at (123.0, 76.0)
- added Q14: Q_NMOS_GDS, TO_SOT_Packages_SMD:TO-252-2, F.Cu at (123.0, 85.0)
- added Q15: Q_NMOS_GDS, TO_SOT_Packages_SMD:TO-252-2, F.Cu at (123.0, 94.0)
- Q2, Q5, Q8: value Q_PMOS_GSD -> Q_NMOS_GSD
- R14: value 18K -> 1K
Connections:
- net Net-(Q1-Pad1) renamed A+G
- net Net-(Q3-Pad1) renamed A-G
- net Net-(Q4-Pad1) renamed B+G
- net Net-(Q6-Pad1) renamed B-G
- net Net-(Q7-Pad1) renamed C+G
- net Net-(Q9-Pad1) renamed C-G
Routing:
- net +12V: track 103.5 -> 228.9 mm
- net B+G: track 2.67 -> 105.4 mm, vias 0 -> 2
- net GND: track 256.9 -> 346.9 mm, vias 6 -> 11
- net C+G: track 2.67 -> 54.8 mm, vias 0 -> 2
- net A+G: track 2.67 -> 40.0 mm
- net B-G: track 14.9 -> 48.1 mm, vias 0 -> 4
- net C: track 72.3 -> 103.7 mm, vias 2 -> 6
- net C-G: track 15.4 -> 45.3 mm, vias 0 -> 4
- net B: track 45.2 -> 73.4 mm, vias 1 -> 5
- net A-G: track 14.6 -> 42.6 mm, vias 0 -> 2
- net A: track 75.8 -> 95.8 mm
- net P13: track 46.9 -> 48.4 mm
- added copper zone on B.Cu, net B
- added copper zone on F.Cu, net B
- added copper zone on B.Cu, net C
- added copper zone on F.Cu, net C
Other:
- board size 65 x 50 mm -> 85 x 60 mm
- board text added: "A+"
- board text added: "A-"
- board text added: "B+"
- board text added: "B-"
- board text added: "BLDC_STC15W408AS 20180706 v0.2"
- board text added: "C+"
- board text added: "C-"
- board text removed: "BLDC 20180622"
