File: KiCAD/BLDC_STC15W401.sch (KiCad schematic (older format))
At the start: 55 parts, among them J1 Download, J2 PPM, J3 BLDC, J4 DC12V, J5 DC5V, J6 PWM, J7 BLDC, Q1 DTC143Z, Q2 Q_PMOS_GSD, Q3 Q_NMOS_GSD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

Commit message: 添加V0.2的PCB设计
Parts:
- removed Q2, Q5, Q8: Q_PMOS_GSD, TO_SOT_Packages_SMD:SOT-23_Handsoldering, symbol Q_PMOS_GSD
- added Q10, Q11, Q12, Q13, Q14, Q15: Q_NMOS_GDS, TO_SOT_Packages_SMD:TO-252-2, symbol Q_NMOS_GDS
- added Q2, Q5, Q8: Q_NMOS_GSD, TO_SOT_Packages_SMD:SOT-23_Handsoldering, symbol Q_NMOS_GSD
- R10, R14, R3: value 18K -> 1K
Connections:
- net +12V: now also Q10.2 (D), Q12.2 (D), Q14.2 (D), Q2.3 (D), Q5.3 (D), Q8.3 (D)
- net A: now also Q10.3 (S), Q11.2 (D), Q2.2 (S)
- net B: now also Q12.3 (S), Q13.2 (D), Q5.2 (S)
- net C: now also Q14.3 (S), Q15.2 (D), Q8.2 (S)
- net GND: now also Q11.3 (S), Q13.3 (S), Q15.3 (S)
- net at Q1.3 (C), R4.2: now also Q2.1 (G)
- net A+G: now reaches Q1.1 (B), R1.1
- net A+G: now also Q10.1 (G)
- net A-G: now reaches Q3.1 (G), R2.1, R3.2
- net A-G: now also Q11.1 (G)
- net at Q4.3 (C), R11.2: now also Q5.1 (G)
- net B+G: now reaches Q4.1 (B), R7.1
- net B+G: now also Q12.1 (G)
- net B-G: now reaches Q6.1 (G), R10.2, R8.1
- net B-G: now also Q13.1 (G)
- net at Q7.3 (C), R16.2: now also Q8.1 (G)
- net C+G: now reaches Q7.1 (B), R12.1
- net C+G: now also Q14.1 (G)
- net C-G: now reaches Q9.1 (G), R13.1, R14.2
- net C-G: now also Q15.1 (G)
